File: ESP32/Smart Home Energy Management System/Smart Home Energy Management System.kicad_pcb (KiCad board)
At the start: 4 copper layers, 198.1 x 130.8 mm, 141 parts, among them J1 NEPA, J10 N, J11 PZEM_SIG, J14 USB_C Conn, J15 TRANS 1-OUT, J17 TRANS-IN, J18 TRANS 2-OUT, J19 DISPLAY, J2 INVERTER, J20 LOAD 6, J21 LOAD 5, J22 LOAD 4, J23 LOAD 3, J24 LOAD 2, J25 LOAD 1, J3 CT, J6 PZEM_LOAD, K1 10A RELAY, K10 30A RELAY, K11 30A RELAY, K12 30A RELAY, K13 30A RELAY, K2 30A RELAY, K3 30A RELAY, K4 30A RELAY, K5 30A RELAY, K6 30A RELAY, K7 30A RELAY, K8 30A RELAY, K9 30A RELAY, Q1 UMH3N, Q2 UMH3N, Q3 ULN2803ADWR, Q4 ULN2803ADWR, SW1 RESET, SW2 FLASH, U1 LM2596S-3.3V, U2 LM2596S-12, U3 ESP32-WROOM, U4 LM2596S-5V, U5 AMS1117-3.3, U6 PCA9555D, U7 CH340C, Y1 12MHz

Commit message: update from work
Other:
- board text added: "JSITECH jsitech4@gmail.com 08133520374"
Changed lines of the file:
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@@
+		)
+	)
+	(gr_text "JSITECH\njsitech4@gmail.com\n08133520374"
+		(at 145.835 70.42 0)
+		(layer "B.SilkS")
+		(effects
+			(font
+				(size 4 2)
+				(thickness 0.5)
+				(bold yes)
+			)
+			(justify bottom mirror)
 		)
 	)
