File: ESP32/Vibration_and_Temperature_Monitoring_System_for_Rotary_Equipment/hardware/Predictive_Maintenance_System_for_Industrial_Motor.kicad_sch (KiCad schematic)
At the start: 75 parts, among them J1 Screw_Terminal_01x03, J10 MPU6050, J2 Screw_Terminal_01x08, J3 OLED SCREEN, J4 LOAD, J5 220VAC, J6 MPU6050, J8 USB_C Conn, J9 12VAC, K1 FINDER-36.11, Q1 UMH3N, SW1 RotaryEncoder, SW2 RESET, SW3 FLASH, U1 AMS1117-3.3, U2 ESP32-S3-WROOM-1U-N16R8, U3 LM2596S-3.3V, U4 LM2596S-5V, U5 CH340C, Y1 12MHz

Commit message: update from work
Parts:
- J10: value MPU6050 -> ADXL345 2
- J2: value Screw_Terminal_01x08 -> MAX31865
- J6: value MPU6050 -> ADXL345 1
- SW1: now left out of the parts list
Changed lines of the file:
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@@
 		(body_style 1)
 		(exclude_from_sim no)
-		(in_bom yes)
+		(in_bom no)
 		(on_board yes)
 		(in_pos_files yes)
@@
 			)
 		)
-		(property "Value" "MPU6050"
+		(property "Value" "ADXL345 1"
 			(at 373.38 304.8001 0)
 			(hide yes)
@@
 			)
 		)
-		(property "Value" "Screw_Terminal_01x08"
+		(property "Value" "MAX31865"
 			(at 384.81 182.8799 0)
 			(hide yes)
@@
 			)
 		)
-		(property "Value" "MPU6050"
+		(property "Value" "ADXL345 2"
 			(at 406.4 304.8001 0)
 			(hide yes)
