File: ESP32/Vibration_and_Temperature_Monitoring_System_for_Rotary_Equipment/hardware/Vibration_and_Temperature_Monitoring_System_for_Rotary_Equipment.kicad_sch (KiCad schematic)
At the start: 77 parts, among them J1 Screw_Terminal_01x03, J2 Screw_Terminal_01x08, J3 OLED SCREEN, J4 LOAD, J5 220VAC, J6 Ultra Sonic, J8 USB_C Conn, J9 12VAC, K1 FINDER-36.11, Q1 UMH3N, SW1 RotaryEncoder, SW2 RESET, SW3 FLASH, U1 AMS1117-3.3, U2 ESP32-S3-WROOM-1U-N16R8, U3 LM2596S-3.3V, U4 LM2596S-5V, U5 CH340C, Y1 12MHz

Commit message: updates from work
Parts:
- removed C26: 100nF, Capacitor_SMD:C_0805_2012Metric_Pad1.18x1.45mm_HandSolder, symbol PCM_SL_Capacitors:104_Ceramic
- removed J6: Ultra Sonic, Connector_PinSocket_2.54mm:PinSocket_1x04_P2.54mm_Vertical, symbol Connector:Screw_Terminal_01x04
- removed R17: 1k, Resistor_SMD:R_0805_2012Metric, symbol PCM_SL_Resistors:10k
- removed R18: 2k, Resistor_SMD:R_0805_2012Metric, symbol PCM_SL_Resistors:10k
- added J10: ADXL345 2, Connector_PinHeader_2.54mm:PinHeader_1x08_P2.54mm_Vertical, symbol Connector:Screw_Terminal_01x08
- added J6: ADXL345 1, Connector_PinHeader_2.54mm:PinHeader_1x08_P2.54mm_Vertical, symbol Connector:Screw_Terminal_01x08
- J2: value Screw_Terminal_01x08 -> MAX31865
- SW1: now left out of the parts list
Connections:
- net +3.3V: now also J10.2 (Pin_2), J6.2 (Pin_2)
- net GND: now also J10.1 (Pin_1), J6.1 (Pin_1)
- net INT1: now also J10.4 (Pin_4), J6.4 (Pin_4)
- net SCL: now also J10.8 (Pin_8), J6.8 (Pin_8)
- net SDA: now also J10.7 (Pin_7), J6.7 (Pin_7)
- new net INT2: J10.5 (Pin_5), J6.5 (Pin_5)
- new net SD0: J10.6 (Pin_6), J6.6 (Pin_6)
- new net VCS: J10.3 (Pin_3), J6.3 (Pin_3)
- no-connect marks 21 -> 27
Other:
- note added: "1"
- note added: "2"
- note added: "ADXL345"
- note added: "MAX31865 MODULE"
- note added: "MOTOR"
- note added: "VIBRATION SENSOR"
- note removed: "PUMP"
- note removed: "TEMPERATURE SENSOR"
- note removed: "ULTRASONIC SENSOR"
- moved on the sheet: BZ1, C10, C11, C12, C13, C14, C15, C16, C17, C18, C19, C2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
