File: ESP32/Hot_Liquid_Monitoring_and_Control_ System/hardware/Hot_Liquid_Monitoring_and_Control_ System.kicad_sch (KiCad schematic)
At the start: 75 parts, among them J1 Screw_Terminal_01x03, J10 ADXL345 2, J2 MAX31865, J3 OLED SCREEN, J4 LOAD, J5 220VAC, J6 ADXL345 1, J8 USB_C Conn, J9 12VAC, K1 FINDER-36.11, Q1 UMH3N, SW1 RotaryEncoder, SW2 RESET, SW3 FLASH, U1 AMS1117-3.3, U2 ESP32-S3-WROOM-1U-N16R8, U3 LM2596S-3.3V, U4 LM2596S-5V, U5 CH340C, Y1 12MHz

Commit message: updates from work
Parts:
- removed J10: ADXL345 2, Connector_PinHeader_2.54mm:PinHeader_1x08_P2.54mm_Vertical, symbol Connector:Screw_Terminal_01x08
- removed J6: ADXL345 1, Connector_PinHeader_2.54mm:PinHeader_1x08_P2.54mm_Vertical, symbol Connector:Screw_Terminal_01x08
- added C26: 100nF, Capacitor_SMD:C_0805_2012Metric_Pad1.18x1.45mm_HandSolder, symbol PCM_SL_Capacitors:104_Ceramic
- added J6: Ultra Sonic, Connector_PinSocket_2.54mm:PinSocket_1x04_P2.54mm_Vertical, symbol Connector:Screw_Terminal_01x04
- added R17: 1k, Resistor_SMD:R_0805_2012Metric, symbol PCM_SL_Resistors:10k
- added R18: 2k, Resistor_SMD:R_0805_2012Metric, symbol PCM_SL_Resistors:10k
- J2: value MAX31865 -> Screw_Terminal_01x08
- SW1: now in the parts list
Connections:
- net +5V: now also C26.2, J6.1 (Pin_1)
- net GND: now also C26.1, J6.4 (Pin_4), R18.1
- net GPIO1: now also R17.2, R18.2
- net GPIO4: now also J6.2 (Pin_2)
- new net: J6.3 (Pin_3), R17.1
- no-connect marks 27 -> 21
Other:
- note added: "PUMP"
- note added: "TEMPERATURE SENSOR"
- note added: "ULTRASONIC SENSOR"
- note removed: "1"
- note removed: "2"
- note removed: "ADXL345"
- note removed: "MAX31865 MODULE"
- note removed: "MOTOR"
- note removed: "VIBRATION SENSOR"
- moved on the sheet: BZ1, C10, C11, C12, C13, C14, C15, C16, C17, C18, C19, C2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
